File: PCB/PCB.kicad_pcb (KiCad board)
At the start: 2 copper layers, 80 x 39.5 mm, 41 parts, among them SW1 KH-6X6X6H-STM, SW2 KH-6X6X6H-STM, SW3 KH-6X6X6H-STM, T1 AO3400A, T2 AO3400A, T3 AO3400A, T4 AO3400A, T5 AO3400A, T6 AO3400A, T7 AO3400A

Commit message: Removed Company Name
Other:
- board text added: "${TITLE}, Rev ${REVISION}"
- board text removed: "${TITLE}, Rev ${REVISION} ${COMPANY}"
Changed lines of the file:
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@@
 			)
 		)
-		(sheetname "Stammblatt")
+		(sheetname "Root")
 		(sheetfile "PCB.kicad_sch")
 		(attr through_hole)
@@
 			)
 		)
-		(sheetname "Stammblatt")
+		(sheetname "Root")
 		(sheetfile "PCB.kicad_sch")
 		(attr smd)
@@
 			)
 		)
-		(sheetname "Stammblatt")
+		(sheetname "Root")
 		(sheetfile "PCB.kicad_sch")
 		(attr smd)
@@
 			)
 		)
-		(sheetname "Stammblatt")
+		(sheetname "Root")
 		(sheetfile "PCB.kicad_sch")
 		(attr smd)
@@
 			)
 		)
-		(sheetname "Stammblatt")
+		(sheetname "Root")
 		(sheetfile "PCB.kicad_sch")
 		(attr through_hole)
@@
 			)
 		)
-		(sheetname "Stammblatt")
+		(sheetname "Root")
 		(sheetfile "PCB.kicad_sch")
 		(attr smd)
@@
 			)
 		)
-		(sheetname "Stammblatt")
+		(sheetname "Root")
 		(sheetfile "PCB.kicad_sch")
 		(attr smd)
@@
 			)
 		)
-		(sheetname "Stammblatt")
+		(sheetname "Root")
 		(sheetfile "PCB.kicad_sch")
 		(attr smd)
@@
 			)
 		)
-		(sheetname "Stammblatt")
+		(sheetname "Root")
 		(sheetfile "PCB.kicad_sch")
 		(attr smd)
@@
 			)
 		)
-		(sheetname "Stammblatt")
+		(sheetname "Root")
 		(sheetfile "PCB.kicad_sch")
 		(attr through_hole)
@@
 			)
 		)
-		(sheetname "Stammblatt")
+		(sheetname "Root")
 		(sheetfile "PCB.kicad_sch")
 		(attr through_hole)
@@
 			)
 		)
-		(sheetname "Stammblatt")
+		(sheetname "Root")
 		(sheetfile "PCB.kicad_sch")
 		(attr through_hole)
@@
 			)
 		)
-		(sheetname "Stammblatt")
+		(sheetname "Root")
 		(sheetfile "PCB.kicad_sch")
 		(attr through_hole)
@@
 			)
 		)
-		(sheetname "Stammblatt")
+		(sheetname "Root")
 		(sheetfile "PCB.kicad_sch")
 		(attr through_hole)
@@
 			)
 		)
-		(sheetname "Stammblatt")
+		(sheetname "Root")
 		(sheetfile "PCB.kicad_sch")
 		(attr smd)
@@
 			)
 		)
-		(sheetname "Stammblatt")
+		(sheetname "Root")
 		(sheetfile "PCB.kicad_sch")
 		(attr smd)
@@
 			)
 		)
-		(sheetname "Stammblatt")
+		(sheetname "Root")
 		(sheetfile "PCB.kicad_sch")
 		(attr through_hole)
@@
 			)
 		)
-		(sheetname "Stammblatt")
+		(sheetname "Root")
 		(sheetfile "PCB.kicad_sch")
 		(attr smd)
@@
 			)
 		)
-		(sheetname "Stammblatt")
+		(sheetname "Root")
 		(sheetfile "PCB.kicad_sch")
 		(attr smd)
@@
 			)
 		)
-		(sheetname "Stammblatt")
+		(sheetname "Root")
 		(sheetfile "PCB.kicad_sch")
 		(attr smd)
@@
 		)
 		(property ki_fp_filters "Choke_* *Coil* Inductor_* L_*")
-		(sheetname "Stammblatt")
+		(sheetname "Root")
 		(sheetfile "PCB.kicad_sch")
 		(attr smd)
@@
 			)
 		)
-		(sheetname "Stammblatt")
+		(sheetname "Root")
 		(sheetfile "PCB.kicad_sch")
 		(attr through_hole)
@@
 			)
 		)
-		(sheetname "Stammblatt")
+		(sheetname "Root")
 		(sheetfile "PCB.kicad_sch")
 		(attr smd)
@@
 			)
 		)
-		(sheetname "Stammblatt")
+		(sheetname "Root")
 		(sheetfile "PCB.kicad_sch")
 		(attr smd)
@@
 			)
 		)
-		(sheetname "Stammblatt")
+		(sheetname "Root")
 		(sheetfile "PCB.kicad_sch")
 		(attr smd)
@@
 			)
 		)
-		(sheetname "Stammblatt")
+		(sheetname "Root")
 		(sheetfile "PCB.kicad_sch")
 		(attr smd)
@@
 			)
 		)
-		(sheetname "Stammblatt")
+		(sheetname "Root")
 		(sheetfile "PCB.kicad_sch")
 		(attr smd)
@@
 			)
 		)
-		(sheetname "Stammblatt")
+		(sheetname "Root")
 		(sheetfile "PCB.kicad_sch")
 		(attr through_hole)
@@
 			)
 		)
-		(sheetname "Stammblatt")
+		(sheetname "Root")
 		(sheetfile "PCB.kicad_sch")
 		(attr through_hole)
@@
 			)
 		)
-		(sheetname "Stammblatt")
+		(sheetname "Root")
 		(sheetfile "PCB.kicad_sch")
 		(attr through_hole)
@@
 			)
 		)
-		(sheetname "Stammblatt")
+		(sheetname "Root")
 		(sheetfile "PCB.kicad_sch")
 		(attr smd)
@@
 			)
 		)
-		(sheetname "Stammblatt")
+		(sheetname "Root")
 		(sheetfile "PCB.kicad_sch")
 		(attr smd)
@@
 			)
 		)
-		(sheetname "Stammblatt")
+		(sheetname "Root")
 		(sheetfile "PCB.kicad_sch")
 		(attr through_hole)
@@
 			)
 		)
-		(sheetname "Stammblatt")
+		(sheetname "Root")
 		(sheetfile "PCB.kicad_sch")
 		(attr smd)
@@
 			)
 		)
-		(sheetname "Stammblatt")
+		(sheetname "Root")
 		(sheetfile "PCB.kicad_sch")
 		(attr smd)
@@
 			)
 		)
-		(sheetname "Stammblatt")
+		(sheetname "Root")
 		(sheetfile "PCB.kicad_sch")
 		(attr smd)
@@
 			)
 		)
-		(sheetname "Stammblatt")
+		(sheetname "Root")
 		(sheetfile "PCB.kicad_sch")
 		(attr smd)
@@
 			)
 		)
-		(sheetname "Stammblatt")
+		(sheetname "Root")
 		(sheetfile "PCB.kicad_sch")
 		(attr through_hole)
@@
 			)
 		)
-		(sheetname "Stammblatt")
+		(sheetname "Root")
 		(sheetfile "PCB.kicad_sch")
 		(attr smd)
@@
 			)
 		)
-		(sheetname "Stammblatt")
+		(sheetname "Root")
 		(sheetfile "PCB.kicad_sch")
 		(attr smd)
@@
 			)
 		)
-		(sheetname "Stammblatt")
+		(sheetname "Root")
 		(sheetfile "PCB.kicad_sch")
 		(attr smd)
@@
 		(layer "Edge.Cuts")
 	)
-	(gr_text "${TITLE}, Rev ${REVISION}\n${COMPANY}"
+	(gr_text "${TITLE}, Rev ${REVISION}\n"
 		(at 62 56 0)
 		(layer "F.SilkS")
