File: PCB/PCB.kicad_sch (KiCad schematic)
At the start: 41 parts, among them SW1 KH-6X6X6H-STM, SW2 KH-6X6X6H-STM, SW3 KH-6X6X6H-STM, T1 AO3400A, T2 AO3400A, T3 AO3400A, T4 AO3400A, T5 AO3400A, T6 AO3400A, T7 AO3400A

Commit message: Removed Company Name
Other:
- company: 2SimpleEnergy GmbH -> (none)
- title: ESP Heating Fan Controller -> Smart Heating Fan Controller
Changed lines of the file:
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@@
 	(paper "A4")
 	(title_block
-		(title "ESP Heating Fan Controller")
+		(title "Smart Heating Fan Controller")
 		(date "2025-01")
 		(rev "1.0")
-		(company "2SimpleEnergy GmbH")
 	)
 	(junction
